Commit message: Imported upstream version '2.3.2' of 'upstream'

File: urdf/camera/OS1-64.urdf.xacro (robot description, xacro)
@@ -24,5 +24,5 @@
          <origin xyz="0 0 0.0" rpy="0 0 1.5707" />
          <geometry>
-           <mesh filename="$(find pal_urdf_utils)/meshes/camera/os1_64.dae" />
+           <mesh filename="package://pal_urdf_utils/meshes/camera/os1_64.dae" />
            <!-- <cylinder length="0.073" radius="0.04" /> -->
          </geometry>

File: urdf/camera/elp_rgb.urdf.xacro (robot description, xacro)
@@ -32,5 +32,5 @@
         <origin xyz="0 0 0" rpy="0 90 0"/>
         <geometry>
-          <mesh filename="$(find pal_urdf_utils)/meshes/camera/elp_camera.stl" scale="0.001 0.001 0.001"/>
+          <mesh filename="package://pal_urdf_utils/meshes/camera/elp_camera.stl" scale="0.001 0.001 0.001"/>
         </geometry>
         <material name="Grey" />

File: urdf/camera/orbbec_astra_pro.urdf.xacro (robot description, xacro)
@@ -35,5 +35,5 @@
         <origin xyz="0 0 0" rpy="0 0 0"/>
         <geometry>
-          <mesh filename="$(find pal_urdf_utils)/meshes/camera/orbbec.STL" />
+          <mesh filename="package://pal_urdf_utils/meshes/camera/orbbec.STL" />
         </geometry>
         <material name="DarkGrey">

File: urdf/camera/rpi_camera.gazebo.xacro (robot description, xacro)
@@ -9,4 +9,5 @@
 <robot xmlns:xacro="http://ros.org/wiki/xacro">
   <xacro:macro name="rpi_camera_gazebo" params="name:=camera topic:=camera frame:=camera_optic_frame">
+    <xacro:include filename="$(find pal_urdf_utils)/urdf/pi.urdf.xacro" />
     <gazebo reference="${name}_link">
       <sensor type="camera" name="${name}_pi_camera">

File: urdf/camera/structure_sensor.urdf.xacro (robot description, xacro)
@@ -34,5 +34,5 @@
         <origin xyz="0 0 0" rpy="0 0 0"/>
         <geometry>
-          <mesh filename="$(find pal_urdf_utils)/meshes/camera/structure_sensor.stl" scale="0.001 0.001 0.001" />
+          <mesh filename="package://pal_urdf_utils/meshes/camera/structure_sensor.stl" scale="0.001 0.001 0.001" />
         </geometry>
         <material name="Grey">

File: urdf/ft_sensors/ati.urdf.xacro (robot description, xacro)
@@ -31,5 +31,5 @@
         <origin xyz="0 0 0" rpy="0 0 0" />
         <geometry>
-          <mesh filename="$(find pal_urdf_utils)/meshes/ft_sensors/ati_ft_sensor.stl"/>
+          <mesh filename="package://pal_urdf_utils//meshes/ft_sensors/ati_ft_sensor.stl"/>
         </geometry>
         <material name="pal/DarkGrey"/>

File: urdf/ft_sensors/rokubi.urdf.xacro (robot description, xacro)
@@ -24,5 +24,5 @@
         <origin xyz="0.0 0.0 0.0" rpy="0.0 0.0 0.0"/>
         <geometry>
-          <mesh filename="$(find pal_urdf_utils)/meshes/ft_sensors/rokubi_ft_sensor.stl"/>
+          <mesh filename="package://pal_urdf_utils/meshes/ft_sensors/rokubi_ft_sensor.stl"/>
         </geometry>
         <material name="pal/DarkGrey"/>

File: urdf/laser/hokuyo_urg_04lx_ug01_laser.urdf.xacro (robot description, xacro)
@@ -24,5 +24,5 @@
         <origin xyz="0 0 0" rpy="0 0 0" />
         <geometry>
-          <mesh filename="$(find pal_urdf_utils)/meshes/laser/hokuyo_urg_04lx_ug01.stl"/>
+          <mesh filename="package://pal_urdf_utils/meshes/laser/hokuyo_urg_04lx_ug01.stl"/>
         </geometry>
         <material name="DarkGrey"/>

File: urdf/laser/range.urdf.xacro (robot description, xacro)
@@ -24,5 +24,5 @@
         <origin xyz="0 0 0" rpy="0 0 0" />
         <geometry>
-          <mesh filename="$(find pal_urdf_utils)/meshes/laser/srf05.stl"/>
+          <mesh filename="package://pal_urdf_utils/meshes/laser/srf05.stl"/>
         </geometry>
         <material name="DarkGrey"/>

File: urdf/laser/sick_nanoscan3_laser.urdf.xacro (robot description, xacro)
@@ -33,5 +33,5 @@
         <origin xyz="0 0 0" rpy="0 0 0" />
         <geometry>
-          <mesh filename="package://pmb3_description/meshes/sensors/sick_nanoscan3.stl"/>
+          <mesh filename="package://pal_urdf_utils/meshes/sensors/sick_nanoscan3.stl"/>
         </geometry>
         <material name="DarkGrey"/>

File: urdf/laser/sick_tim551_laser.urdf.xacro (robot description, xacro)
@@ -24,5 +24,5 @@
         <origin xyz="0 0 0" rpy="0 0 0" />
         <geometry>
-          <mesh filename="$(find pal_urdf_utils)/meshes/laser/sick_tim551.stl"/>
+          <mesh filename="package://pal_urdf_utils/meshes/laser/sick_tim551.stl"/>
         </geometry>
         <material name="DarkGrey"/>

File: urdf/laser/sick_tim561_laser.urdf.xacro (robot description, xacro)
@@ -24,5 +24,5 @@
         <origin xyz="0 0 0" rpy="0 0 0" />
         <geometry>
-          <mesh filename="$(find pal_urdf_utils)/meshes/laser/sick_tim551.stl"/>
+          <mesh filename="package://pal_urdf_utils/meshes/laser/sick_tim551.stl"/>
         </geometry>
         <material name="DarkGrey"/>

File: urdf/laser/sick_tim571_laser.urdf.xacro (robot description, xacro)
@@ -24,5 +24,5 @@
         <origin xyz="0 0 0" rpy="0 0 0" />
         <geometry>
-          <mesh filename="$(find pal_urdf_utils)/meshes/laser/sick_tim551.stl"/>
+          <mesh filename="package://pal_urdf_utils/meshes/laser/sick_tim551.stl"/>
         </geometry>
         <material name="DarkGrey"/>

File: urdf/laser/ydlidar_tg15_laser.urdf.xacro (robot description, xacro)
@@ -21,8 +21,14 @@
         <origin xyz="0 0 0" rpy="0 0 0" />
         <geometry>
-          <mesh filename="$(find pal_urdf_utils)/meshes/laser/ydlidar.dae"/>
+          <mesh filename="package://pal_urdf_utils/meshes/laser/ydlidar.dae"/>
         </geometry>
         <material name="DarkGrey"/>
       </visual>
+      <collision>
+        <origin xyz="0 0 0" rpy="0 0 0" />
+        <geometry>
+          <mesh filename="package://pal_urdf_utils/meshes/laser/ydlidar.dae"/>
+        </geometry>
+      </collision>
     </link>
     <joint name="${name}_joint" type="fixed">

File: urdf/laser/ydlidar_tg30_laser.urdf.xacro (robot description, xacro)
@@ -21,8 +21,14 @@
         <origin xyz="0 0 0" rpy="0 0 0" />
         <geometry>
-          <mesh filename="$(find pal_urdf_utils)/meshes/laser/ydlidar.dae"/>
+          <mesh filename="package://pal_urdf_utils/meshes/laser/ydlidar.dae"/>
         </geometry>
         <material name="DarkGrey"/>
       </visual>
+      <collision>
+        <origin xyz="0 0 0" rpy="0 0 0" />
+        <geometry>
+          <mesh filename="package://pal_urdf_utils/meshes/laser/ydlidar.dae"/>
+        </geometry>
+      </collision>
     </link>
     <joint name="${name}_joint" type="fixed">
